File: ProgrammableLM317.sch (KiCad schematic (older format))
At the start: 25 parts, among them IC1 ATTINY85-P, K1 CONN_3, P1 CONN_2, P2 CONN_2, U1 LM317, U2 LM358, U3 MCP4801, U4 7805

Commit message: adding connector to supply negative rail to op amp.
Parts:
- added C5: 0.1uF, ~, symbol C_CER
- added P3: CONN_2, symbol CONN_2
- added R4: 100k, ~, symbol R_0W25_1PCT
Connections:
- net labels added: Vee
- wire segments 86 -> 94
Other:
- moved on the sheet: R1, R2
Changed lines of the file:
@@
 Sheet 1 1
 Title ""
-Date "6 apr 2015"
+Date "8 apr 2015"
 Rev ""
 Comp ""
@@
 L R_0W25_1PCT R1
 U 1 1 550F91CC
-P 8650 5050
-F 0 "R1" V 8730 5050 40  0000 C CNN
-F 1 "10k" V 8657 5051 40  0000 C CNN
-F 2 "~" V 8580 5050 30  0000 C CNN
-F 3 "~" H 8650 5050 30  0000 C CNN
-	1    8650 5050
+P 7150 6350
+F 0 "R1" V 7230 6350 40  0000 C CNN
+F 1 "10k" V 7157 6351 40  0000 C CNN
+F 2 "~" V 7080 6350 30  0000 C CNN
+F 3 "~" H 7150 6350 30  0000 C CNN
+	1    7150 6350
 	-1   0    0    -1
 $EndComp
@@
 L R_0W25_1PCT R2
 U 1 1 550F91DB
-P 8650 5650
-F 0 "R2" V 8730 5650 40  0000 C CNN
-F 1 "33k" V 8657 5651 40  0000 C CNN
-F 2 "~" V 8580 5650 30  0000 C CNN
-F 3 "~" H 8650 5650 30  0000 C CNN
-	1    8650 5650
-	-1   0    0    -1
+P 7900 6000
+F 0 "R2" V 7980 6000 40  0000 C CNN
+F 1 "33k" V 7907 6001 40  0000 C CNN
+F 2 "~" V 7830 6000 30  0000 C CNN
+F 3 "~" H 7900 6000 30  0000 C CNN
+	1    7900 6000
+	0    1    -1   0
 $EndComp
 $Comp
 L GND #PWR02
 U 1 1 550F91EA
-P 7950 5200
-F 0 "#PWR02" H 7950 5200 30  0001 C CNN
-F 1 "GND" H 7950 5130 30  0001 C CNN
-F 2 "" H 7950 5200 60  0000 C CNN
-F 3 "" H 7950 5200 60  0000 C CNN
-	1    7950 5200
-	-1   0    0    -1
+P 7750 5000
+F 0 "#PWR02" H 7750 5000 30  0001 C CNN
+F 1 "GND" H 7750 4930 30  0001 C CNN
+F 2 "" H 7750 5000 60  0000 C CNN
+F 3 "" H 7750 5000 60  0000 C CNN
+	1    7750 5000
+	1    0    0    1
 $EndComp
 $Comp
 L GND #PWR03
 U 1 1 550F9224
-P 8650 6000
-F 0 "#PWR03" H 8650 6000 30  0001 C CNN
-F 1 "GND" H 8650 5930 30  0001 C CNN
-F 2 "" H 8650 6000 60  0000 C CNN
-F 3 "" H 8650 6000 60  0000 C CNN
-	1    8650 6000
+P 7150 6700
+F 0 "#PWR03" H 7150 6700 30  0001 C CNN
+F 1 "GND" H 7150 6630 30  0001 C CNN
+F 2 "" H 7150 6700 60  0000 C CNN
+F 3 "" H 7150 6700 60  0000 C CNN
+	1    7150 6700
 	-1   0    0    -1
 $EndComp
@@
 	6300 1400 6300 1300
 Wire Wire Line
-	7950 5100 7950 5200
-Wire Wire Line
-	8650 4800 8650 4700
-Wire Wire Line
-	8850 4700 8550 4700
-Wire Wire Line
-	8650 5300 8650 5400
-Wire Wire Line
-	8650 5900 8650 6000
-Wire Wire Line
-	8650 5350 7450 5350
-Wire Wire Line
-	7450 5350 7450 4800
+	7950 5100 7950 5600
+Wire Wire Line
+	8650 4700 8650 6000
+Wire Wire Line
+	8550 4700 8850 4700
+Wire Wire Line
+	7450 6000 7450 4800
 Wire Wire Line
 	7450 4800 7550 4800
-Connection ~ 8650 5350
 Wire Wire Line
 	7750 4400 7750 4300
@@
 	7000 1700 7000 2550
 Wire Wire Line
-	8850 2550 8850 4700
+	8850 4700 8850 2550
 Connection ~ 8650 4700
 Wire Wire Line
@@
 Wire Wire Line
 	4250 4750 4250 5050
-Text Notes 9250 5400 2    60   ~ 0
+Text Notes 7000 6050 2    60   ~ 0
 Gain = 4.3
 Text Notes 7500 4550 2    60   ~ 0
@@
 Connection ~ 6400 1400
 $Comp
-L GND #PWR017
+L GND #PWR016
 U 1 1 5512631C
 P 6400 2000
-F 0 "#PWR017" H 6400 2000 30  0001 C CNN
+F 0 "#PWR016" H 6400 2000 30  0001 C CNN
 F 1 "GND" H 6400 1930 30  0001 C CNN
 F 2 "" H 6400 2000 60  0000 C CNN
@@
 $EndComp
 $Comp
-L GND #PWR018
+L GND #PWR017
 U 1 1 5512643D
 P 7950 2000
-F 0 "#PWR018" H 7950 2000 30  0001 C CNN
+F 0 "#PWR017" H 7950 2000 30  0001 C CNN
 F 1 "GND" H 7950 1930 30  0001 C CNN
 F 2 "" H 7950 2000 60  0000 C CNN
@@
 Connection ~ 6650 1400
 Wire Wire Line
-	7000 2550 8850 2550
+	8850 2550 7000 2550
+$Comp
+L CONN_2 P3
+U 1 1 5525B73B
+P 1050 2950
+F 0 "P3" V 1000 2950 40  0000 C CNN
+F 1 "CONN_2" V 1100 2950 40  0000 C CNN
+F 2 "" H 1050 2950 60  0000 C CNN
+F 3 "" H 1050 2950 60  0000 C CNN
+	1    1050 2950
+	-1   0    0    -1
+$EndComp
+$Comp
+L GND #PWR018
+U 1 1 5525B743
+P 1500 2750
+F 0 "#PWR018" H 1500 2750 30  0001 C CNN
+F 1 "GND" H 1500 2680 30  0001 C CNN
+F 2 "" H 1500 2750 60  0000 C CNN
+F 3 "" H 1500 2750 60  0000 C CNN
+	1    1500 2750
+	-1   0    0    1
+$EndComp
+Text GLabel 1500 3150 3    60   Input ~ 0
+Vee
+Wire Wire Line
+	1400 2850 1500 2850
+Wire Wire Line
+	1500 2850 1500 2750
+Wire Wire Line
+	1400 3050 1500 3050
+Wire Wire Line
+	1500 3050 1500 3150
+$Comp
+L C_CER C5
+U 1 1 5525B83E
+P 7750 5300
+F 0 "C5" H 7770 5360 30  0000 L BNN
+F 1 "0.1uF" H 7770 5240 30  0000 L TNN
+F 2 "~" H 7788 5150 30  0000 C CNN
+F 3 "~" H 7750 5300 60  0000 C CNN
+	1    7750 5300
+	-1   0    0    -1
+$EndComp
+Wire Wire Line
+	7750 5100 7750 5000
+Text GLabel 7950 5600 3    60   Input ~ 0
+Vee
+Wire Wire Line
+	7750 5500 7950 5500
+Connection ~ 7950 5500
+$Comp
+L R_0W25_1PCT R4
+U 1 1 5525B9E4
+P 7150 5650
+F 0 "R4" V 7230 5650 40  0000 C CNN
+F 1 "100k" V 7157 5651 40  0000 C CNN
+F 2 "~" V 7080 5650 30  0000 C CNN
+F 3 "~" H 7150 5650 30  0000 C CNN
+	1    7150 5650
+	-1   0    0    -1
+$EndComp
+Wire Wire Line
+	7150 6600 7150 6700
+Wire Wire Line
+	7150 5900 7150 6100
+Text GLabel 7150 5300 1    60   Input ~ 0
+5V
+Wire Wire Line
+	7150 5300 7150 5400
+Wire Wire Line
+	7150 6000 7650 6000
+Connection ~ 7150 6000
+Connection ~ 7450 6000
+Wire Wire Line
+	8650 6000 8150 6000
 $EndSCHEMATC
